File: bvm-a-card-breakout.sch (KiCad schematic (older format))
At the start: 6 parts, among them J1 mezz-conn-02x50, J2 mezz-conn-02x50, J3 Conn_01x25, J4 Conn_01x25, J5 Conn_01x25, J6 Conn_01x25

Commit message: Fixed slight misalignment in connector footprints
Parts:
- J1: footprint TX25-100P-LT-H1E:TX24-100R-LT-H1E -> TX25-100P-LT-H1E:TX25-100P-LT-H1E
Changed lines of the file:
@@
 LIBS:valves
 LIBS:mezz-conn-02x50
+LIBS:bvm-a-card-breakout-cache
 EELAYER 25 0
 EELAYER END
@@
 F 0 "J1" V 8100 5250 60  0000 C CNN
 F 1 "mezz-conn-02x50" V 450 5250 60  0000 C CNN
-F 2 "TX25-100P-LT-H1E:TX24-100R-LT-H1E" H 4150 5250 60  0001 C CNN
+F 2 "TX25-100P-LT-H1E:TX25-100P-LT-H1E" H 4150 5250 60  0001 C CNN
 F 3 "" H 4150 5250 60  0001 C CNN
 	1    4150 5250

Commit message: Updated to full-size Z-board replacement
Parts:
- added J11: mezz-conn-02x50, TX25-100P-LT-H1E:TX25-100P-LT-H1E, symbol mezz-conn-02x50:mezz-conn-02x50
- added J12: mezz-conn-02x50, TX24-100R-LT-H1E:TX24-100R-LT-H1E, symbol mezz-conn-02x50:mezz-conn-02x50
- added J13, J14, J15, J16: Conn_01x25, Connector_PinHeader_2.54mm:PinHeader_1x25_P2.54mm_Vertical, symbol bvm-a-card-breakout-rescue:Conn_01x25
- J1, J2: symbol mezz-conn-02x50 -> mezz-conn-02x50:mezz-conn-02x50
- J3, J4, J5, J6: footprint Pin_Headers:Pin_Header_Straight_1x25_Pitch2.54mm -> Connector_PinHeader_2.54mm:PinHeader_1x25_P2.54mm_Vertical; symbol Conn_01x25 -> bvm-a-card-breakout-rescue:Conn_01x25
Connections:
- new net A10_2: J11.A10, J12.A10, J16.5 (Pin_5)
- new net A11_2: J11.A11, J12.A11, J14.6 (Pin_6)
- new net A12_2: J11.A12, J12.A12, J16.6 (Pin_6)
- new net A13_2: J11.A13, J12.A13, J14.7 (Pin_7)
- new net A14_2: J11.A14, J12.A14, J16.7 (Pin_7)
- new net A15_2: J11.A15, J12.A15, J14.8 (Pin_8)
- new net A16_2: J11.A16, J12.A16, J16.8 (Pin_8)
- new net A17_2: J11.A17, J12.A17, J14.9 (Pin_9)
- new net A18_2: J11.A18, J12.A18, J16.9 (Pin_9)
- new net A19_2: J11.A19, J12.A19, J14.10 (Pin_10)
- new net A1_2: J11.A1, J12.A1, J14.1 (Pin_1)
- new net A20_2: J11.A20, J12.A20, J16.10 (Pin_10)
- new net A21_2: J11.A21, J12.A21, J14.11 (Pin_11)
- new net A22_2: J11.A22, J12.A22, J16.11 (Pin_11)
- new net A23_2: J11.A23, J12.A23, J14.12 (Pin_12)
- new net A24_2: J11.A24, J12.A24, J16.12 (Pin_12)
- new net A25_2: J11.A25, J12.A25, J14.13 (Pin_13)
- new net A26_2: J11.A26, J12.A26, J16.13 (Pin_13)
- new net A27_2: J11.A27, J12.A27, J14.14 (Pin_14)
- new net A28_2: J11.A28, J12.A28, J16.14 (Pin_14)
- new net A29_2: J11.A29, J12.A29, J14.15 (Pin_15)
- new net A2_2: J11.A2, J12.A2, J16.1 (Pin_1)
- new net A30_2: J11.A30, J12.A30, J16.15 (Pin_15)
- new net A31_2: J11.A31, J12.A31, J14.16 (Pin_16)
- new net A32_2: J11.A32, J12.A32, J16.16 (Pin_16)
- new net A33_2: J11.A33, J12.A33, J14.17 (Pin_17)
- new net A34_2: J11.A34, J12.A34, J16.17 (Pin_17)
- new net A35_2: J11.A35, J12.A35, J14.18 (Pin_18)
- new net A36_2: J11.A36, J12.A36, J16.18 (Pin_18)
- new net A37_2: J11.A37, J12.A37, J14.19 (Pin_19)
- new net A38_2: J11.A38, J12.A38, J16.19 (Pin_19)
- new net A39_2: J11.A39, J12.A39, J14.20 (Pin_20)
- new net A3_2: J11.A3, J12.A3, J14.2 (Pin_2)
- new net A40_2: J11.A40, J12.A40, J16.20 (Pin_20)
- new net A41_2: J11.A41, J12.A41, J14.21 (Pin_21)
- new net A42_2: J11.A42, J12.A42, J16.21 (Pin_21)
- new net A43_2: J11.A43, J12.A43, J14.22 (Pin_22)
- new net A44_2: J11.A44, J12.A44, J16.22 (Pin_22)
- new net A45_2: J11.A45, J12.A45, J14.23 (Pin_23)
- new net A46_2: J11.A46, J12.A46, J16.23 (Pin_23)
- new net A47_2: J11.A47, J12.A47, J14.24 (Pin_24)
- new net A48_2: J11.A48, J12.A48, J16.24 (Pin_24)
- new net A49_2: J11.A49, J12.A49, J14.25 (Pin_25)
- new net A4_2: J11.A4, J12.A4, J16.2 (Pin_2)
- new net A50_2: J11.A50, J12.A50, J16.25 (Pin_25)
- new net A5_2: J11.A5, J12.A5, J14.3 (Pin_3)
- new net A6_2: J11.A6, J12.A6, J16.3 (Pin_3)
- new net A7_2: J11.A7, J12.A7, J14.4 (Pin_4)
- new net A8_2: J11.A8, J12.A8, J16.4 (Pin_4)
- new net A9_2: J11.A9, J12.A9, J14.5 (Pin_5)
- new net B10_2: J11.B10, J12.B10, J15.5 (Pin_5)
- new net B11_2: J11.B11, J12.B11, J13.6 (Pin_6)
- new net B12_2: J11.B12, J12.B12, J15.6 (Pin_6)
- new net B13_2: J11.B13, J12.B13, J13.7 (Pin_7)
- new net B14_2: J11.B14, J12.B14, J15.7 (Pin_7)
- new net B15_2: J11.B15, J12.B15, J13.8 (Pin_8)
- new net B16_2: J11.B16, J12.B16, J15.8 (Pin_8)
- new net B17_2: J11.B17, J12.B17, J13.9 (Pin_9)
- new net B18_2: J11.B18, J12.B18, J15.9 (Pin_9)
- new net B19_2: J11.B19, J12.B19, J13.10 (Pin_10)
- new net B1_2: J11.B1, J12.B1, J13.1 (Pin_1)
- new net B20_2: J11.B20, J12.B20, J15.10 (Pin_10)
- new net B21_2: J11.B21, J12.B21, J13.11 (Pin_11)
- new net B22_2: J11.B22, J12.B22, J15.11 (Pin_11)
- new net B23_2: J11.B23, J12.B23, J13.12 (Pin_12)
- new net B24_2: J11.B24, J12.B24, J15.12 (Pin_12)
- new net B25_2: J11.B25, J12.B25, J13.13 (Pin_13)
- new net B26_2: J11.B26, J12.B26, J15.13 (Pin_13)
- new net B27_2: J11.B27, J12.B27, J13.14 (Pin_14)
- new net B28_2: J11.B28, J12.B28, J15.14 (Pin_14)
- new net B29_2: J11.B29, J12.B29, J13.15 (Pin_15)
- new net B2_2: J11.B2, J12.B2, J15.1 (Pin_1)
- new net B30_2: J11.B30, J12.B30, J15.15 (Pin_15)
- new net B31_2: J11.B31, J12.B31, J13.16 (Pin_16)
- new net B32_2: J11.B32, J12.B32, J15.16 (Pin_16)
- new net B33_2: J11.B33, J12.B33, J13.17 (Pin_17)
- new net B34_2: J11.B34, J12.B34, J15.17 (Pin_17)
- new net B35_2: J11.B35, J12.B35, J13.18 (Pin_18)
- new net B36_2: J11.B36, J12.B36, J15.18 (Pin_18)
- new net B37_2: J11.B37, J12.B37, J13.19 (Pin_19)
- new net B38_2: J11.B38, J12.B38, J15.19 (Pin_19)
- new net B39_2: J11.B39, J12.B39, J13.20 (Pin_20)
- new net B3_2: J11.B3, J12.B3, J13.2 (Pin_2)
- new net B40_2: J11.B40, J12.B40, J15.20 (Pin_20)
- new net B41_2: J11.B41, J12.B41, J13.21 (Pin_21)
- new net B42_2: J11.B42, J12.B42, J15.21 (Pin_21)
- new net B43_2: J11.B43, J12.B43, J13.22 (Pin_22)
- new net B44_2: J11.B44, J12.B44, J15.22 (Pin_22)
- new net B45_2: J11.B45, J12.B45, J13.23 (Pin_23)
- new net B46_2: J11.B46, J12.B46, J15.23 (Pin_23)
- new net B47_2: J11.B47, J12.B47, J13.24 (Pin_24)
- new net B48_2: J11.B48, J12.B48, J15.24 (Pin_24)
- new net B49_2: J11.B49, J12.B49, J13.25 (Pin_25)
- new net B4_2: J11.B4, J12.B4, J15.2 (Pin_2)
- new net B50_2: J11.B50, J12.B50, J15.25 (Pin_25)
- new net B5_2: J11.B5, J12.B5, J13.3 (Pin_3)
- new net B6_2: J11.B6, J12.B6, J15.3 (Pin_3)
- new net B7_2: J11.B7, J12.B7, J13.4 (Pin_4)
- new net B8_2: J11.B8, J12.B8, J15.4 (Pin_4)
- new net B9_2: J11.B9, J12.B9, J13.5 (Pin_5)
Other:
- moved on the sheet: J1, J2, J3, J4, J5, J6
